Commit message: consolidated cx_descriptions to one package; fixed the isu_lab.xacro to be accurate

File: Automated-Grinding/JDH/jdh_ws_cx/src/khi_cx_description/urdf/cx.urdf.xacro (robot description, xacro)
@@ -1,8 +1,11 @@
 <?xml version="1.0" ?>
-<robot name="khi_cx165l" xmlns:xacro="http://ros.org/wiki/xacro">
+<robot name="khi_cx" xmlns:xacro="http://ros.org/wiki/xacro">
   <xacro:include filename="$(find khi_cx_description)/urdf/cx165l_macro.xacro"/>
+  <xacro:include filename="$(find khi_cx_description)/urdf/cx110l_macro.xacro"/>
   <!-- instantiate cx165l -->
   <xacro:khi_cx165l prefix="" />
-  <!-- Fix both cx robots to world -->
+    <!-- instantiate cx110l -->
+  <xacro:khi_cx110l prefix="" />
+  <!-- Fix cx165l to world -->
   <link name="world"/>
   <joint name="world2base_cx165l" type="fixed">
@@ -14,5 +17,5 @@
     <parent link="world"/>
     <child link="base_plate_cx110l"/>
-    <origin rpy="0 0 0" xyz="-5.0546 0 0"/>
+    <origin rpy="0 0 0" xyz="0 0 0"/>
   </joint>
 </robot>

File: Automated-Grinding/JDH/jdh_ws_cx/src/khi_cx_description/urdf/cx110l.urdf.xacro (robot description, xacro)
@@ -1,7 +1,7 @@
 <?xml version="1.0" ?>
-<robot name="khi_cx165l" xmlns:xacro="http://ros.org/wiki/xacro">
-  <xacro:include filename="$(find khi_cx_description)/urdf/cx165l_macro.xacro"/>
-  <!-- instantiate cx165l -->
-  <xacro:khi_cx165l prefix="" />
+<robot name="khi_cx110l" xmlns:xacro="http://ros.org/wiki/xacro">
+  <xacro:include filename="$(find khi_cx_description)/urdf/cx110l_macro.xacro"/>
+  <!-- instantiate cx110l -->
+  <xacro:khi_cx110l prefix="" />
   <!-- Fix both cx robots to world -->
   <link name="world"/>

File: Automated-Grinding/JDH/jdh_ws_cx/src/khi_cx_description/urdf/cx110l_macro.xacro (robot description, xacro)
@@ -2,7 +2,7 @@
 <robot xmlns:xacro="http://ros.org/wiki/xacro">
   <xacro:macro name="khi_cx110l" params="prefix">
-    <xacro:include filename="$(find khi_cx110l_description)/urdf/cx.transmission.xacro" />
-    <xacro:include filename="$(find khi_cx110l_description)/urdf/common.gazebo.xacro" />
-    <xacro:include filename="$(find khi_cx110l_description)/urdf/isu_lab.xacro" />
+    <xacro:include filename="$(find khi_cx_description)/urdf/cx.transmission.xacro" />
+    <xacro:include filename="$(find khi_cx_description)/urdf/common.gazebo.xacro" />
+    <xacro:include filename="$(find khi_cx_description)/urdf/isu_lab.xacro" />
     <!-- link rviz colors -->
     <material name="White">
@@ -49,5 +49,5 @@
     </xacro:macro>
     <joint name="${prefix}base_link_joint" type="fixed">
-        <parent link="base_plate" />
+        <parent link="base_plate_cx110l" />
         <child link="base_link" />
         <origin rpy="0 0 0" xyz="0 0 0" />
@@ -61,19 +61,19 @@
             <geometry>
                 <mesh
-                filename="package://khi_cx110l_description/meshes/CX165L-BASE.STL" />
-            </geometry>
-            <material
-                name="">
-                <color
-                rgba="0.75294 0.75294 0.75294 1" />
-            </material>
-        </visual>
-        <collision>
-            <origin
-                xyz="0 0 0"
-                rpy="0 0 0" />
-            <geometry>
-                <mesh
-                filename="package://khi_cx110l_description/meshes/CX165L-BASE-HULL.STL" />
+                filename="package://khi_cx_description/cx110l_meshes/CX165L-BASE.STL" />
+            </geometry>
+            <material
+                name="">
+                <color
+                rgba="0.75294 0.75294 0.75294 1" />
+            </material>
+        </visual>
+        <collision>
+            <origin
+                xyz="0 0 0"
+                rpy="0 0 0" />
+            <geometry>
+                <mesh
+                filename="package://khi_cx_description/cx110l_meshes/CX165L-BASE-HULL.STL" />
             </geometry>
         </collision>
@@ -96,19 +96,19 @@
             <geometry>
                 <mesh
-                filename="package://khi_cx110l_description/meshes/CX165L-J1.STL"/>
-            </geometry>
-            <material
-                name="">
-                <color
-                rgba="0.75294 0.75294 0.75294 1" />
-            </material>
-        </visual>
-        <collision>
-            <origin
-                xyz="0 0 0"
-                rpy="0 0 0" />
-            <geometry>
-                <mesh
-                filename="package://khi_cx110l_description/meshes/CX165L-J1-HULL.STL" />
+                filename="package://khi_cx_description/cx110l_meshes/CX165L-J1.STL"/>
+            </geometry>
+            <material
+                name="">
+                <color
+                rgba="0.75294 0.75294 0.75294 1" />
+            </material>
+        </visual>
+        <collision>
+            <origin
+                xyz="0 0 0"
+                rpy="0 0 0" />
+            <geometry>
+                <mesh
+                filename="package://khi_cx_description/cx110l_meshes/CX165L-J1-HULL.STL" />
             </geometry>
         </collision>
@@ -131,19 +131,19 @@
             <geometry>
                 <mesh
-                filename="package://khi_cx110l_description/meshes/CX165L-J2.STL" />
-            </geometry>
-            <material
-                name="">
-                <color
-                rgba="0.75294 0.75294 0.75294 1" />
-            </material>
-        </visual>
-        <collision>
-            <origin
-                xyz="0 0 0"
-                rpy="0 0 0" />
-            <geometry>
-                <mesh
-                filename="package://khi_cx110l_description/meshes/CX165L-J2-HULL.STL" />
+                filename="package://khi_cx_description/cx110l_meshes/CX165L-J2.STL" />
+            </geometry>
+            <material
+                name="">
+                <color
+                rgba="0.75294 0.75294 0.75294 1" />
+            </material>
+        </visual>
+        <collision>
+            <origin
+                xyz="0 0 0"
+                rpy="0 0 0" />
+            <geometry>
+                <mesh
+                filename="package://khi_cx_description/cx110l_meshes/CX165L-J2-HULL.STL" />
             </geometry>
         </collision>
@@ -166,19 +166,19 @@
             <geometry>
                 <mesh
-                filename="package://khi_cx110l_description/meshes/CX165L-J3.STL" />
-            </geometry>
-            <material
-                name="">
-                <color
-                rgba="0.75294 0.75294 0.75294 1" />
-            </material>
-        </visual>
-        <collision>
-            <origin
-                xyz="0 0 0"
-                rpy="0 0 0" />
-            <geometry>
-                <mesh
-                filename="package://khi_cx110l_description/meshes/CX165L-J3-HULL.STL" />
+                filename="package://khi_cx_description/cx110l_meshes/CX165L-J3.STL" />
+            </geometry>
+            <material
+                name="">
+                <color
+                rgba="0.75294 0.75294 0.75294 1" />
+            </material>
+        </visual>
+        <collision>
+            <origin
+                xyz="0 0 0"
+                rpy="0 0 0" />
+            <geometry>
+                <mesh
+                filename="package://khi_cx_description/cx110l_meshes/CX165L-J3-HULL.STL" />
             </geometry>
         </collision>
@@ -201,5 +201,5 @@
             <geometry>
                 <mesh
-                filename="package://khi_cx110l_description/meshes/CX165L-J4.STL"  />
+                filename="package://khi_cx_description/cx110l_meshes/CX165L-J4.STL"  />
             </geometry>
             <material
@@ -215,5 +215,5 @@
             <geometry>
                 <mesh
-                filename="package://khi_cx110l_description/meshes/CX165L-J4-HULL.STL"  />
+                filename="package://khi_cx_description/cx110l_meshes/CX165L-J4-HULL.STL"  />
             </geometry>
         </collision>
@@ -236,19 +236,19 @@
             <geometry>
                 <mesh
-                filename="package://khi_cx110l_description/meshes/CX165L-J5.STL" />
-            </geometry>
-            <material
-                name="">
-                <color
-                rgba="0.75294 0.75294 0.75294 1" />
-            </material>
-        </visual>
-        <collision>
-            <origin
-                xyz="0 0 0"
-                rpy="0 0 0" />
-            <geometry>
-                <mesh
-                filename="package://khi_cx110l_description/meshes/CX165L-J5-HULL.STL"/>
+                filename="package://khi_cx_description/cx110l_meshes/CX165L-J5.STL" />
+            </geometry>
+            <material
+                name="">
+                <color
+                rgba="0.75294 0.75294 0.75294 1" />
+            </material>
+        </visual>
+        <collision>
+            <origin
+                xyz="0 0 0"
+                rpy="0 0 0" />
+            <geometry>
+                <mesh
+                filename="package://khi_cx_description/cx110l_meshes/CX165L-J5-HULL.STL"/>
             </geometry>
         </collision>
@@ -271,19 +271,19 @@
             <geometry>
                 <mesh
-                filename="package://khi_cx110l_description/meshes/CX165L-J6.STL" />
-            </geometry>
-            <material
-                name="">
-                <color
-                rgba="0.75294 0.75294 0.75294 1" />
-            </material>
-        </visual>
-        <collision>
-            <origin
-                xyz="0 0 0"
-                rpy="0 0 0" />
-            <geometry>
-                <mesh
-                filename="package://khi_cx110l_description/meshes/CX165L-J6-HULL.STL" />
+                filename="package://khi_cx_description/cx110l_meshes/CX165L-J6.STL" />
+            </geometry>
+            <material
+                name="">
+                <color
+                rgba="0.75294 0.75294 0.75294 1" />
+            </material>
+        </visual>
+        <collision>
+            <origin
+                xyz="0 0 0"
+                rpy="0 0 0" />
+            <geometry>
+                <mesh
+                filename="package://khi_cx_description/cx110l_meshes/CX165L-J6-HULL.STL" />
             </geometry>
         </collision>

File: Automated-Grinding/JDH/jdh_ws_cx/src/khi_cx_description/urdf/cx165l_macro.xacro (robot description, xacro)
@@ -49,5 +49,5 @@
     </xacro:macro>
     <joint name="${prefix}base_link_joint" type="fixed">
-        <parent link="base_plate" />
+        <parent link="base_plate_cx165l" />
         <child link="base_link" />
         <origin rpy="0 0 0" xyz="0 0 0" />
@@ -61,19 +61,19 @@
             <geometry>
                 <mesh
-                filename="package://khi_cx_description/meshes/CX165L-BASE.STL" />
-            </geometry>
-            <material
-                name="">
-                <color
-                rgba="0.75294 0.75294 0.75294 1" />
-            </material>
-        </visual>
-        <collision>
-            <origin
-                xyz="0 0 0"
-                rpy="0 0 0" />
-            <geometry>
-                <mesh
-                filename="package://khi_cx_description/meshes/CX165L-BASE-HULL.STL" />
+                filename="package://khi_cx_description/cx165l_meshes/CX165L-BASE.STL" />
+            </geometry>
+            <material
+                name="">
+                <color
+                rgba="0.75294 0.75294 0.75294 1" />
+            </material>
+        </visual>
+        <collision>
+            <origin
+                xyz="0 0 0"
+                rpy="0 0 0" />
+            <geometry>
+                <mesh
+                filename="package://khi_cx_description/cx165l_meshes/CX165L-BASE-HULL.STL" />
             </geometry>
         </collision>
@@ -96,19 +96,19 @@
             <geometry>
                 <mesh
-                filename="package://khi_cx_description/meshes/CX165L-J1.STL"/>
-            </geometry>
-            <material
-                name="">
-                <color
-                rgba="0.75294 0.75294 0.75294 1" />
-            </material>
-        </visual>
-        <collision>
-            <origin
-                xyz="0 0 0"
-                rpy="0 0 0" />
-            <geometry>
-                <mesh
-                filename="package://khi_cx_description/meshes/CX165L-J1-HULL.STL" />
+                filename="package://khi_cx_description/cx165l_meshes/CX165L-J1.STL"/>
+            </geometry>
+            <material
+                name="">
+                <color
+                rgba="0.75294 0.75294 0.75294 1" />
+            </material>
+        </visual>
+        <collision>
+            <origin
+                xyz="0 0 0"
+                rpy="0 0 0" />
+            <geometry>
+                <mesh
+                filename="package://khi_cx_description/cx165l_meshes/CX165L-J1-HULL.STL" />
             </geometry>
         </collision>
@@ -131,19 +131,19 @@
             <geometry>
                 <mesh
-                filename="package://khi_cx_description/meshes/CX165L-J2.STL" />
-            </geometry>
-            <material
-                name="">
-                <color
-                rgba="0.75294 0.75294 0.75294 1" />
-            </material>
-        </visual>
-        <collision>
-            <origin
-                xyz="0 0 0"
-                rpy="0 0 0" />
-            <geometry>
-                <mesh
-                filename="package://khi_cx_description/meshes/CX165L-J2-HULL.STL" />
+                filename="package://khi_cx_description/cx165l_meshes/CX165L-J2.STL" />
+            </geometry>
+            <material
+                name="">
+                <color
+                rgba="0.75294 0.75294 0.75294 1" />
+            </material>
+        </visual>
+        <collision>
+            <origin
+                xyz="0 0 0"
+                rpy="0 0 0" />
+            <geometry>
+                <mesh
+                filename="package://khi_cx_description/cx165l_meshes/CX165L-J2-HULL.STL" />
             </geometry>
         </collision>
@@ -166,19 +166,19 @@
             <geometry>
                 <mesh
-                filename="package://khi_cx_description/meshes/CX165L-J3.STL" />
-            </geometry>
-            <material
-                name="">
-                <color
-                rgba="0.75294 0.75294 0.75294 1" />
-            </material>
-        </visual>
-        <collision>
-            <origin
-                xyz="0 0 0"
-                rpy="0 0 0" />
-            <geometry>
-                <mesh
-                filename="package://khi_cx_description/meshes/CX165L-J3-HULL.STL" />
+                filename="package://khi_cx_description/cx165l_meshes/CX165L-J3.STL" />
+            </geometry>
+            <material
+                name="">
+                <color
+                rgba="0.75294 0.75294 0.75294 1" />
+            </material>
+        </visual>
+        <collision>
+            <origin
+                xyz="0 0 0"
+                rpy="0 0 0" />
+            <geometry>
+                <mesh
+                filename="package://khi_cx_description/cx165l_meshes/CX165L-J3-HULL.STL" />
             </geometry>
         </collision>
@@ -201,5 +201,5 @@
             <geometry>
                 <mesh
-                filename="package://khi_cx_description/meshes/CX165L-J4.STL"  />
+                filename="package://khi_cx_description/cx165l_meshes/CX165L-J4.STL"  />
             </geometry>
             <material
@@ -215,5 +215,5 @@
             <geometry>
                 <mesh
-                filename="package://khi_cx_description/meshes/CX165L-J4-HULL.STL"  />
+                filename="package://khi_cx_description/cx165l_meshes/CX165L-J4-HULL.STL"  />
             </geometry>
         </collision>
@@ -236,19 +236,19 @@
             <geometry>
                 <mesh
-                filename="package://khi_cx_description/meshes/CX165L-J5.STL" />
-            </geometry>
-            <material
-                name="">
-                <color
-                rgba="0.75294 0.75294 0.75294 1" />
-            </material>
-        </visual>
-        <collision>
-            <origin
-                xyz="0 0 0"
-                rpy="0 0 0" />
-            <geometry>
-                <mesh
-                filename="package://khi_cx_description/meshes/CX165L-J5-HULL.STL"/>
+                filename="package://khi_cx_description/cx165l_meshes/CX165L-J5.STL" />
+            </geometry>
+            <material
+                name="">
+                <color
+                rgba="0.75294 0.75294 0.75294 1" />
+            </material>
+        </visual>
+        <collision>
+            <origin
+                xyz="0 0 0"
+                rpy="0 0 0" />
+            <geometry>
+                <mesh
+                filename="package://khi_cx_description/cx165l_meshes/CX165L-J5-HULL.STL"/>
             </geometry>
         </collision>
@@ -271,19 +271,19 @@
             <geometry>
                 <mesh
-                filename="package://khi_cx_description/meshes/CX165L-J6.STL" />
-            </geometry>
-            <material
-                name="">
-                <color
-                rgba="0.75294 0.75294 0.75294 1" />
-            </material>
-        </visual>
-        <collision>
-            <origin
-                xyz="0 0 0"
-                rpy="0 0 0" />
-            <geometry>
-                <mesh
-                filename="package://khi_cx_description/meshes/CX165L-J6-HULL.STL" />
+                filename="package://khi_cx_description/cx165l_meshes/CX165L-J6.STL" />
+            </geometry>
+            <material
+                name="">
+                <color
+                rgba="0.75294 0.75294 0.75294 1" />
+            </material>
+        </visual>
+        <collision>
+            <origin
+                xyz="0 0 0"
+                rpy="0 0 0" />
+            <geometry>
+                <mesh
+                filename="package://khi_cx_description/cx165l_meshes/CX165L-J6-HULL.STL" />
             </geometry>
         </collision>
@@ -303,19 +303,19 @@
             <geometry>
                 <mesh
-                filename="package://khi_cx_description/meshes/CX165L-PUSHCORP.STL" />
-            </geometry>
-            <material
-                name="">
-                <color
-                rgba="0.75294 0.75294 0.75294 1" />
-            </material>
-        </visual>
-        <collision>
-            <origin
-                xyz="0 0 0"
-                rpy="0 0 0" />
-            <geometry>
-                <mesh
-                filename="package://khi_cx_description/meshes/CX165L-PUSHCORP-HULL.STL" />
+                filename="package://khi_cx_description/cx165l_meshes/CX165L-PUSHCORP.STL" />
+            </geometry>
+            <material
+                name="">
+                <color
+                rgba="0.75294 0.75294 0.75294 1" />
+            </material>
+        </visual>
+        <collision>
+            <origin
+                xyz="0 0 0"
+                rpy="0 0 0" />
+            <geometry>
+                <mesh
+                filename="package://khi_cx_description/cx165l_meshes/CX165L-PUSHCORP-HULL.STL" />
             </geometry>
         </collision>
