Commit message: consolidated cx_descriptions to one package; fixed the isu_lab.xacro to be accurate

File: Automated-Grinding/JDH/jdh_ws_cx/src/khi_cx_description/urdf/isu_lab.xacro (robot description, xacro)
@@ -9,5 +9,5 @@
     </xacro:macro>
     <!-- Lab Environment -->
-     <link name="base_plate">
+    <link name="base_plate_cx165l">
         <visual>
             <origin
@@ -33,4 +33,28 @@
         <xacro:default_inertial mass="1"/>
     </link>
+    <link name="base_plate_cx110l">
+        <visual>
+            <origin
+                xyz="0 0 0.0127"
+                rpy="0 0 0" />
+            <geometry>
+                <box size="1.016 1.016 0.0254" />
+            </geometry>
+            <material
+                name="">
+                <color
+                rgba="0.75294 0.75294 0.75294 1" />
+            </material>
+        </visual>
+        <collision>
+            <origin
+                xyz="0 0 4.0"
+                rpy="0 0 0" />
+            <geometry>
+                <box size="1.016 1.016 0.0254" />
+            </geometry>
+        </collision>
+        <xacro:default_inertial mass="1"/>
+    </link>
     <joint name="world2east_wall" type="fixed">
         <parent link="world"/>
@@ -41,21 +65,21 @@
         <visual>
             <origin
-                xyz="-0.7888 -0.7612 2.5"
-                rpy="0 0 0" />
-            <geometry>
-                <box size="3 0.1 5" />
-            </geometry>
-            <material
-                name="">
-                <color
-                rgba="0.75294 0.75294 0.75294 1" />
-            </material>
-        </visual>
-        <collision>
-            <origin
-                xyz="-0.7888 -0.7612 2.5"
-                rpy="0 0 0" />
-            <geometry>
-                <box size="3 0.1 5" />
+                xyz="-2.53 -0.81 2.5"
+                rpy="0 0 0" />
+            <geometry>
+                <box size="6.68 0.1 5" />
+            </geometry>
+            <material
+                name="">
+                <color
+                rgba="0.75294 0.75294 0.75294 1" />
+            </material>
+        </visual>
+        <collision>
+            <origin
+                xyz="-2.53 -0.81 2.5"
+                rpy="0 0 0" />
+            <geometry>
+                <box size="6.68 0.1 5" />
             </geometry>
         </collision>
@@ -70,21 +94,21 @@
         <visual>
             <origin
-                xyz="3.7612 0.9398 0.5"
-                rpy="0 0 0" />
-            <geometry>
-                <box size="0.1 3.302 1" />
-            </geometry>
-            <material
-                name="">
-                <color
-                rgba="0.75294 0.75294 0.75294 1" />
-            </material>
-        </visual>
-        <collision>
-            <origin
-                xyz="3.7612 0.9398 0.5"
-                rpy="0 0 0" />
-            <geometry>
-                <box size="0.1 3.302 5" />
+                xyz="0.810 1.717 2.5"
+                rpy="0 0 0" />
+            <geometry>
+                <box size="0.1 5.055 5" />
+            </geometry>
+            <material
+                name="">
+                <color
+                rgba="0.75294 0.75294 0.75294 1" />
+            </material>
+        </visual>
+        <collision>
+            <origin
+                xyz="0.810 1.717 0.5"
+                rpy="0 0 0" />
+            <geometry>
+                <box size="0.1 5.055 5" />
             </geometry>
         </collision>
@@ -99,21 +123,21 @@
         <visual>
             <origin
-                xyz="0 0 -0.05"
-                rpy="0 0 0" />
-            <geometry>
-                <box size="6 6 0.1" />
-            </geometry>
-            <material
-                name="">
-                <color
-                rgba="0.75294 0.75294 0.75294 1" />
-            </material>
-        </visual>
-        <collision>
-            <origin
-                xyz="0 0 -0.05"
-                rpy="0 0 0" />
-            <geometry>
-                <box size="6 6 0.1" />
+                xyz="-2.53 1.717 -0.063"
+                rpy="0 0 0" />
+            <geometry>
+                <box size="6.68 5.055 0.1" />
+            </geometry>
+            <material
+                name="">
+                <color
+                rgba="0.75294 0.75294 0.75294 1" />
+            </material>
+        </visual>
+        <collision>
+            <origin
+                xyz="-2.53 1.717 -0.063"
+                rpy="0 0 0" />
+            <geometry>
+                <box size="6.68 5.055 0.1" />
             </geometry>
         </collision>
@@ -128,21 +152,21 @@
         <visual>
             <origin
-                xyz="-0.7888 2.6392 2.5"
-                rpy="0 0 0" />
-            <geometry>
-                <box size="3 0.1 5" />
-            </geometry>
-            <material
-                name="">
-                <color
-                rgba="0.75294 0.75294 0.75294 0.2" />
-            </material>
-        </visual>
-        <collision>
-            <origin
-                xyz="-0.7888 2.6392 2.5"
-                rpy="0 0 0" />
-            <geometry>
-                <box size="3 0.1 5" />
+                xyz="-2.53 4.245 2.5"
+                rpy="0 0 0" />
+            <geometry>
+                <box size="6.68 0.1 5" />
+            </geometry>
+            <material
+                name="">
+                <color
+                rgba="0.75294 0.75294 0.75294 0.1" />
+            </material>
+        </visual>
+        <collision>
+            <origin
+                xyz="-2.53 4.245 2.5"
+                rpy="0 0 0" />
+            <geometry>
+                <box size="6.68 0.1 5" />
             </geometry>
         </collision>
@@ -157,21 +181,21 @@
         <visual>
             <origin
-                xyz="-2.3344 0.9398 2.5"
-                rpy="0 0 0" />
-            <geometry>
-                <box size="0.1 3.302 5" />
-            </geometry>
-            <material
-                name="">
-                <color
-                rgba="0.75294 0.75294 0.75294 0.2" />
-            </material>
-        </visual>
-        <collision>
-            <origin
-                xyz="-2.3344 0.9398 2.5"
-                rpy="0 0 0" />
-            <geometry>
-                <box size="0.1 3.302 5" />
+                xyz="-5.878 1.7175 2.5"
+                rpy="0 0 0" />
+            <geometry>
+                <box size="0.1 5.055 5" />
+            </geometry>
+            <material
+                name="">
+                <color
+                rgba="0.75294 0.75294 0.75294 0.1" />
+            </material>
+        </visual>
+        <collision>
+            <origin
+                xyz="-5.878 1.7175 2.5"
+                rpy="0 0 0" />
+            <geometry>
+                <box size="0.1 5.055 5" />
             </geometry>
         </collision>
