Commit message: Made changes to MTC

File: Automated-Grinding/WWG/wwg_ws_cx/src/khi_cx_description/urdf/cx110l_macro.xacro (robot description, xacro)
@@ -22,23 +22,23 @@
     <xacro:property name="j6_mass" value="3"/>
     <!-- joint limits [rad] -->
-    <xacro:property name="j1_lower_limit" value="${radians(0)}"/>
-    <xacro:property name="j1_upper_limit" value="${radians(90)}"/>
-    <xacro:property name="j2_lower_limit" value="${radians(-36)}"/>
-    <xacro:property name="j2_upper_limit" value="${radians( 80)}"/>
-    <xacro:property name="j3_lower_limit" value="${radians(-75)}"/>
-    <xacro:property name="j3_upper_limit" value="${radians( 0)}"/>
-    <xacro:property name="j4_lower_limit" value="${radians(-210)}"/>
-    <xacro:property name="j4_upper_limit" value="${radians( 210)}"/>
-    <xacro:property name="j5_lower_limit" value="${radians(-120)}"/>
-    <xacro:property name="j5_upper_limit" value="${radians( 120)}"/>
+    <xacro:property name="j1_lower_limit" value="${radians(-360)}"/>
+    <xacro:property name="j1_upper_limit" value="${radians(360)}"/>
+    <xacro:property name="j2_lower_limit" value="${radians(-360)}"/>
+    <xacro:property name="j2_upper_limit" value="${radians(360)}"/>
+    <xacro:property name="j3_lower_limit" value="${radians(-360)}"/>
+    <xacro:property name="j3_upper_limit" value="${radians(360)}"/>
+    <xacro:property name="j4_lower_limit" value="${radians(-360)}"/>
+    <xacro:property name="j4_upper_limit" value="${radians(360)}"/>
+    <xacro:property name="j5_lower_limit" value="${radians(-360)}"/>
+    <xacro:property name="j5_upper_limit" value="${radians(360)}"/>
     <xacro:property name="j6_lower_limit" value="${radians(-360)}"/>
-    <xacro:property name="j6_upper_limit" value="${radians( 360)}"/>
+    <xacro:property name="j6_upper_limit" value="${radians(6.28319)}"/>
     <!-- joint velocity limits [rad/s] -->
-    <xacro:property name="j1_velocity_limit" value="${radians(130)}"/>
-    <xacro:property name="j2_velocity_limit" value="${radians(125)}"/>
-    <xacro:property name="j3_velocity_limit" value="${radians(125)}"/>
-    <xacro:property name="j4_velocity_limit" value="${radians(180)}"/>
-    <xacro:property name="j5_velocity_limit" value="${radians(180)}"/>
-    <xacro:property name="j6_velocity_limit" value="${radians(280)}"/>
+    <xacro:property name="j1_velocity_limit" value="${radians(360)}"/>
+    <xacro:property name="j2_velocity_limit" value="${radians(360)}"/>
+    <xacro:property name="j3_velocity_limit" value="${radians(360)}"/>
+    <xacro:property name="j4_velocity_limit" value="${radians(360)}"/>
+    <xacro:property name="j5_velocity_limit" value="${radians(360)}"/>
+    <xacro:property name="j6_velocity_limit" value="${radians(360)}"/>
     <!-- link inertial(TODO : set correct link inertial )-->
     <xacro:macro name="default_inertial" params="mass">
